File: hw/sns_node.kicad_pcb (KiCad board)
At the start: 2 copper layers, 0 parts

Commit message: - update schematic and place comps
Parts:
- added C1: 4.7uF, SM0402, F.Cu at (202.9, 112.8)
- added C2: 10uF, SM0402, F.Cu at (218.7, 112.8)
- added C3: 1uF, SM0402, F.Cu at (213.5, 112.8)
- added C4: 1uF, SM0402, F.Cu at (211.7, 112.8)
- added J1: USB-MICRO-B, usb_micro_b_smt, F.Cu at (217.9, 99.7)
- added J2: ARM_10PIN, ARM_10_PIN_SMT, F.Cu at (205.6, 105.5)
- added JP1: JUMPER, jmp_small, F.Cu at (217.0, 110.2)
- added P1: BATT-, TEST_0.100, F.Cu at (226.3, 109.6)
- added P2: BATT+, TEST_0.100, F.Cu at (224.4, 109.6)
- added P3: +3.3v, TEST_0.100, F.Cu at (218.8, 109.6)
- added P4: SCL, TEST_0.100, F.Cu at (228.2, 109.6)
- added P5: GND, TEST_0.100, F.Cu at (222.6, 109.6)
- added P6: SDA, TEST_0.100, F.Cu at (220.7, 109.6)
- added Q1: MOSFET_N, SOT23, F.Cu at (207.9, 110.5)
- added Q2: MOSFET_P, SOT23, F.Cu at (211.2, 110.5)
- added Q3: MOSFET_N, SOT23, F.Cu at (214.5, 110.5)
- added R1: 3M, SM0402, F.Cu at (206.5, 112.8)
- added R10: 3M, SM0402, F.Cu at (222.2, 112.8)
- added R11: 3M, SM0402, F.Cu at (204.7, 112.8)
- added R3: 3M, SM0402, F.Cu at (225.7, 112.8)
- added R4: 1M, SM0402, F.Cu at (220.5, 112.8)
- added R5: 1.3M, SM0402, F.Cu at (215.3, 112.8)
- added R6: 240K, SM0402, F.Cu at (216.9, 112.8)
- added R7: 510K, SM0402, F.Cu at (223.9, 112.8)
- added R8: 100K, SM0402, F.Cu at (208.3, 112.8)
- added R9: 100K, SM0402, F.Cu at (209.9, 112.8)
- added SW1: SW_PUSH, spst_pushbutton_smd, F.Cu at (203.2, 96.6)
- added U1: INDUCTOR, CDRH4D18C_inductor, F.Cu at (210.4, 103.5)
- added U2: MCP1640_SOT23, MCP1640, F.Cu at (226.2, 105.8)
- added U3: SI7020, si7020_dfn6, F.Cu at (202.7, 109.2)
- added U4: MKL02ZXVFG4, MKL02_QFN16, F.Cu at (217.8, 105.3)
- added U5: AAT3220_SC-59-3, sc59, F.Cu at (224.8, 104.3)
- added U6: NRF24L01_MOD_HDR, nrf24_8pin, F.Cu at (224.4, 99.1)
