File: hw/sns_node.sch (KiCad schematic (older format))
At the start: 28 parts, among them J1 USB-MICRO-B, J2 ARM_10PIN, P1 BATT-, P2 BATT+, Q1 MOSFET_P, Q2 MOSFET_N, SW1 SW_PUSH, U1 SI7020, U2 INDUCTOR, U3 MCP1640_SOT23, U4 MKL02ZXVFG4, U5 NRF24L01_MOD_HDR, U6 AAT3220_SC-59-3

Commit message: - add header for connecting i2c daughter boards - add acc_pwr fet
Parts:
- added JP?: JUMPER, ~, symbol JUMPER
- added P? (x4): TST, ~, symbol TST
- added Q?: MOSFET_N, ~, symbol MOSFET_N
- added R?: 3M, ~, symbol R
Connections:
- net labels added: ACC_PWR, ACC_PWR_CTRL, NRF_PWR_CTRL
- net labels removed: NRF_PWR_CRTL, TEMP_SNS_PWR
- wire segments 90 -> 101
Other:
- moved on the sheet: C?, Q1, Q?, R1, R5, R6, R?

Commit message: - remove power-on circuit, pullup OK because IO keeps state during micro sleep.
Parts:
- removed C?: 4.7uF, ~, symbol C
- removed Q?: MOSFET_P, ~, symbol MOSFET_P
- removed R?: 1M, ~, symbol R
- added R1, R2: 3M, ~, symbol R
- gave numbers to parts that had none: 7
- renumbered Q1 to Q2, Q2 to Q3, R7 to R10, R8 to R11, R1 to R4, R2 to R5, R3 to R6, R4 to R7, R5 to R8, R6 to R9, U2 to U1, U3 to U2, U1 to U3, U6 to U5, U5 to U6
Connections:
- net labels added: SWITCH/VBUS_SNS
- net labels removed: SWITCH
Other:
- note added: "NP- accessory\nexpansion\nheader"
- note added: "NP- optional accessory\npower control"
- note added: "weak pullup to\nstart LPS. I/O\nstates are preserved\nthrough sleep mode."
- moved on the sheet: JP1, P1, P2, P3, P4, P5, P6, Q1, Q2, Q3, R10, R11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

Commit message: - new kicadlib, associations.
Parts:
- removed R2: 3M, ~, symbol R
- P3: value TST -> +3.3v
- P4: value TST -> SCL
- P5: value TST -> GND
- P6: value TST -> SDA
Connections:
- wire segments 101 -> 98
Changed lines of the file:
@@
 Sheet 1 1
 Title ""
-Date "27 feb 2014"
+Date "8 mar 2014"
 Rev ""
 Comp ""
@@
 $EndComp
 $Comp
-L GND #PWR3
+L GND #PWR01
 U 1 1 5302BFFF
 P 1850 2650
-F 0 "#PWR3" H 1850 2650 30  0001 C CNN
+F 0 "#PWR01" H 1850 2650 30  0001 C CNN
 F 1 "GND" H 1850 2580 30  0001 C CNN
 F 2 "" H 1850 2650 60  0000 C CNN
@@
 	1850 2300 1850 2650
 Wire Wire Line
-	1350 2450 1950 2450
+	1550 2450 1950 2450
 $Comp
 L INDUCTOR U1
@@
 BATT+
 $Comp
-L GND #PWR6
+L GND #PWR02
 U 1 1 5302C089
 P 3400 2100
-F 0 "#PWR6" H 3400 2100 30  0001 C CNN
+F 0 "#PWR02" H 3400 2100 30  0001 C CNN
 F 1 "GND" H 3400 2030 30  0001 C CNN
 F 2 "" H 3400 2100 60  0000 C CNN
@@
 $EndComp
 $Comp
-L GND #PWR7
+L GND #PWR03
 U 1 1 5302C0E1
 P 3400 4150
-F 0 "#PWR7" H 3400 4150 30  0001 C CNN
+F 0 "#PWR03" H 3400 4150 30  0001 C CNN
 F 1 "GND" H 3400 4080 30  0001 C CNN
 F 2 "" H 3400 4150 60  0000 C CNN
@@
 $EndComp
 $Comp
-L GND #PWR8
+L GND #PWR04
 U 1 1 5302C147
 P 3850 2800
-F 0 "#PWR8" H 3850 2800 30  0001 C CNN
+F 0 "#PWR04" H 3850 2800 30  0001 C CNN
 F 1 "GND" H 3850 2730 30  0001 C CNN
 F 2 "" H 3850 2800 60  0000 C CNN
@@
 	850  1050 950  1050
 Connection ~ 3050 1600
-Text GLabel 1350 2450 0    60   Input ~ 0
+Text GLabel 1550 2450 0    60   Input ~ 0
 EN
 $Comp
-L GND #PWR9
+L GND #PWR05
 U 1 1 5302C467
 P 4850 4200
-F 0 "#PWR9" H 4850 4200 30  0001 C CNN
+F 0 "#PWR05" H 4850 4200 30  0001 C CNN
 F 1 "GND" H 4850 4130 30  0001 C CNN
 F 2 "" H 4850 4200 60  0000 C CNN
@@
 	2150 3200 2150 3300
 $Comp
-L GND #PWR4
+L GND #PWR06
 U 1 1 5302C99C
 P 2150 4500
-F 0 "#PWR4" H 2150 4500 30  0001 C CNN
+F 0 "#PWR06" H 2150 4500 30  0001 C CNN
 F 1 "GND" H 2150 4430 30  0001 C CNN
 F 2 "" H 2150 4500 60  0000 C CNN
@@
 Connection ~ 7000 1250
 $Comp
-L GND #PWR11
+L GND #PWR07
 U 1 1 53055869
 P 7000 1950
-F 0 "#PWR11" H 7000 1950 30  0001 C CNN
+F 0 "#PWR07" H 7000 1950 30  0001 C CNN
 F 1 "GND" H 7000 1880 30  0001 C CNN
 F 2 "" H 7000 1950 60  0000 C CNN
@@
 	7000 1950 7000 1850
 $Comp
-L GND #PWR15
+L GND #PWR08
 U 1 1 530559E5
 P 8750 1050
-F 0 "#PWR15" H 8750 1050 30  0001 C CNN
+F 0 "#PWR08" H 8750 1050 30  0001 C CNN
 F 1 "GND" H 8750 980 30  0001 C CNN
 F 2 "" H 8750 1050 60  0000 C CNN
@@
 SDA
 $Comp
-L GND #PWR5
+L GND #PWR09
 U 1 1 5305676F
 P 3300 7050
-F 0 "#PWR5" H 3300 7050 30  0001 C CNN
+F 0 "#PWR09" H 3300 7050 30  0001 C CNN
 F 1 "GND" H 3300 6980 30  0001 C CNN
 F 2 "" H 3300 7050 60  0000 C CNN
@@
 $EndComp
 $Comp
-L GND #PWR14
+L GND #PWR010
 U 1 1 5305714D
 P 8400 6250
-F 0 "#PWR14" H 8400 6250 30  0001 C CNN
+F 0 "#PWR010" H 8400 6250 30  0001 C CNN
 F 1 "GND" H 8400 6180 30  0001 C CNN
 F 2 "" H 8400 6250 60  0000 C CNN
@@
 	9450 6550 9550 6550
 $Comp
-L GND #PWR17
+L GND #PWR011
 U 1 1 5305785A
 P 9500 6400
-F 0 "#PWR17" H 9500 6400 30  0001 C CNN
+F 0 "#PWR011" H 9500 6400 30  0001 C CNN
 F 1 "GND" H 9500 6330 30  0001 C CNN
 F 2 "" H 9500 6400 60  0000 C CNN
@@
 	8950 3250 9750 3250
 $Comp
-L GND #PWR16
+L GND #PWR012
 U 1 1 530576F0
 P 8950 3850
-F 0 "#PWR16" H 8950 3850 30  0001 C CNN
+F 0 "#PWR012" H 8950 3850 30  0001 C CNN
 F 1 "GND" H 8950 3780 30  0001 C CNN
 F 2 "" H 8950 3850 60  0000 C CNN
@@
 $EndComp
 $Comp
-L GND #PWR13
+L GND #PWR013
 U 1 1 53057711
 P 7850 3900
-F 0 "#PWR13" H 7850 3900 30  0001 C CNN
+F 0 "#PWR013" H 7850 3900 30  0001 C CNN
 F 1 "GND" H 7850 3830 30  0001 C CNN
 F 2 "" H 7850 3900 60  0000 C CNN
@@
 $EndComp
 $Comp
-L GND #PWR12
+L GND #PWR014
 U 1 1 53057717
 P 7850 3100
-F 0 "#PWR12" H 7850 3100 30  0001 C CNN
+F 0 "#PWR014" H 7850 3100 30  0001 C CNN
 F 1 "GND" H 7850 3030 30  0001 C CNN
 F 2 "" H 7850 3100 60  0000 C CNN
@@
 	8950 3750 8950 3850
 $Comp
-L GND #PWR18
+L GND #PWR015
 U 1 1 53057EAB
 P 9650 4100
-F 0 "#PWR18" H 9650 4100 30  0001 C CNN
+F 0 "#PWR015" H 9650 4100 30  0001 C CNN
 F 1 "GND" H 9650 4030 30  0001 C CNN
 F 2 "" H 9650 4100 60  0000 C CNN
@@
 Connection ~ 1700 6300
 $Comp
-L GND #PWR2
+L GND #PWR016
 U 1 1 530BF570
 P 1700 7000
-F 0 "#PWR2" H 1700 7000 30  0001 C CNN
+F 0 "#PWR016" H 1700 7000 30  0001 C CNN
 F 1 "GND" H 1700 6930 30  0001 C CNN
 F 2 "" H 1700 7000 60  0000 C CNN
@@
 P 5600 6650
 F 0 "P3" H 5600 6950 40  0000 C CNN
-F 1 "TST" H 5600 6900 30  0000 C CNN
+F 1 "+3.3v" H 5600 6900 30  0000 C CNN
 F 2 "~" H 5600 6650 60  0000 C CNN
 F 3 "~" H 5600 6650 60  0000 C CNN
@@
 P 5750 6650
 F 0 "P4" H 5750 6950 40  0000 C CNN
-F 1 "TST" H 5750 6900 30  0000 C CNN
+F 1 "SCL" H 5750 6900 30  0000 C CNN
 F 2 "~" H 5750 6650 60  0000 C CNN
 F 3 "~" H 5750 6650 60  0000 C CNN
@@
 P 5900 6650
 F 0 "P5" H 5900 6950 40  0000 C CNN
-F 1 "TST" H 5900 6900 30  0000 C CNN
+F 1 "GND" H 5900 6900 30  0000 C CNN
 F 2 "~" H 5900 6650 60  0000 C CNN
 F 3 "~" H 5900 6650 60  0000 C CNN
@@
 P 6050 6650
 F 0 "P6" H 6050 6950 40  0000 C CNN
-F 1 "TST" H 6050 6900 30  0000 C CNN
+F 1 "SDA" H 6050 6900 30  0000 C CNN
 F 2 "~" H 6050 6650 60  0000 C CNN
 F 3 "~" H 6050 6650 60  0000 C CNN
@@
 SCL
 $Comp
-L GND #PWR10
+L GND #PWR017
 U 1 1 530BF694
 P 5900 6750
-F 0 "#PWR10" H 5900 6750 30  0001 C CNN
+F 0 "#PWR017" H 5900 6750 30  0001 C CNN
 F 1 "GND" H 5900 6680 30  0001 C CNN
 F 2 "" H 5900 6750 60  0000 C CNN
@@
 Text GLabel 7600 6150 0    60   Input ~ 0
 SWITCH/VBUS_SNS
-$Comp
-L R R2
-U 1 1 530F36B4
-P 1550 2100
-F 0 "R2" V 1630 2100 40  0000 C CNN
-F 1 "3M" V 1557 2101 40  0000 C CNN
-F 2 "~" V 1480 2100 30  0000 C CNN
-F 3 "~" H 1550 2100 30  0000 C CNN
-	1    1550 2100
-	1    0    0    -1
-$EndComp
-Wire Wire Line
-	1550 2350 1550 2450
-Connection ~ 1550 2450
-Text GLabel 1450 1750 0    60   Input ~ 0
-BATT+
-Wire Wire Line
-	1550 1850 1550 1750
-Wire Wire Line
-	1550 1750 1450 1750
-Text Notes 500  2000 0    60   ~ 0
+Text Notes 1000 3550 0    60   ~ 0
 weak pullup to\nstart LPS. I/O\nstates are preserved\nthrough sleep mode.
 Wire Wire Line
@@
 $EndComp
 $Comp
-L GND #PWR1
+L GND #PWR018
 U 1 1 530F3C3A
 P 1400 4900
-F 0 "#PWR1" H 1400 4900 30  0001 C CNN
+F 0 "#PWR018" H 1400 4900 30  0001 C CNN
 F 1 "GND" H 1400 4830 30  0001 C CNN
 F 2 "" H 1400 4900 60  0000 C CNN

Commit message: - change vbus sns to share vfb_sns pin. add pdf.
Parts:
- removed Q2: MOSFET_P, ~, symbol MOSFET_P
- added Q2: MOSFET_N, ~, symbol MOSFET_N
- added R?: 10K, ~, symbol R
- added R?: 20K, ~, symbol R
Connections:
- net labels added: USER_SW, VFB_SNS/USB_SNS
- net labels removed: SWITCH/VBUS_SNS
- wire segments 98 -> 104
Other:
- note added: "weak pulldown to\nstart LPS. I/O\nstates are preserved\nthrough sleep mode."
- note removed: "weak pullup to\nstart LPS. I/O\nstates are preserved\nthrough sleep mode."
- moved on the sheet: J2, R11, SW1

Commit message: - update schematic and place comps
Parts:
- removed Q2: MOSFET_N, ~, symbol MOSFET_N
- removed R1: 3M, ~, symbol R
- added R?: 0R, ~, symbol R
Other:
- note added: "nopop"
- note added: "weak pullup to\nstart LPS. I/O\nstates are preserved\nthrough sleep mode."
- note removed: "weak pulldown to\nstart LPS. I/O\nstates are preserved\nthrough sleep mode."
- moved on the sheet: Q3, R10, R4
Changed lines of the file:
@@
 Sheet 1 1
 Title ""
-Date "21 apr 2014"
+Date "24 apr 2014"
 Rev ""
 Comp ""
@@
 Text GLabel 4850 4050 0    60   Input ~ 0
 VCC
-Text GLabel 2400 3900 2    60   Input ~ 0
+Text GLabel 2550 4450 2    60   Input ~ 0
 EN
 $Comp
 L R R4
 U 1 1 5302C818
-P 2150 3550
-F 0 "R4" V 2230 3550 40  0000 C CNN
-F 1 "1M" V 2157 3551 40  0000 C CNN
-F 2 "~" V 2080 3550 30  0000 C CNN
-F 3 "~" H 2150 3550 30  0000 C CNN
-	1    2150 3550
-	1    0    0    -1
-$EndComp
-Text GLabel 1150 4200 0    60   Input ~ 0
+P 2450 4100
+F 0 "R4" V 2530 4100 40  0000 C CNN
+F 1 "1M" V 2457 4101 40  0000 C CNN
+F 2 "~" V 2380 4100 30  0000 C CNN
+F 3 "~" H 2450 4100 30  0000 C CNN
+	1    2450 4100
+	1    0    0    -1
+$EndComp
+Text GLabel 2350 4450 0    60   Input ~ 0
 EN_CTRL
-Text GLabel 2050 3200 0    60   Input ~ 0
+Text GLabel 2350 3750 0    60   Input ~ 0
 BATT+
-$Comp
-L GND #PWR4
-U 1 1 5302C99C
-P 2150 4500
-F 0 "#PWR4" H 2150 4500 30  0001 C CNN
-F 1 "GND" H 2150 4430 30  0001 C CNN
-F 2 "" H 2150 4500 60  0000 C CNN
-F 3 "" H 2150 4500 60  0000 C CNN
-	1    2150 4500
-	1    0    0    -1
-$EndComp
 $Comp
 L 2X4_HDR U6
@@
 Text GLabel 9850 1500 2    60   Input ~ 0
 IRQ
-Text GLabel 7350 1550 2    60   Input ~ 0
+Text GLabel 6600 1750 2    60   Input ~ 0
 NRF_PWR
 $Comp
 L MOSFET_N Q3
 U 1 1 5305557D
-P 7250 1250
-F 0 "Q3" H 7250 1050 60  0000 R CNN
-F 1 "MOSFET_N" H 7250 1450 60  0000 R CNN
-F 2 "~" H 7250 1250 60  0000 C CNN
-F 3 "~" H 7250 1250 60  0000 C CNN
-	1    7250 1250
-	1    0    0    -1
-$EndComp
-Text GLabel 6950 1250 0    60   Input ~ 0
+P 6500 1300
+F 0 "Q3" H 6500 1100 60  0000 R CNN
+F 1 "MOSFET_N" H 6500 1500 60  0000 R CNN
+F 2 "~" H 6500 1300 60  0000 C CNN
+F 3 "~" H 6500 1300 60  0000 C CNN
+	1    6500 1300
+	1    0    0    -1
+$EndComp
+Text GLabel 6200 1300 0    60   Input ~ 0
 NRF_PWR_CTRL
-Text GLabel 7350 950  2    60   Input ~ 0
+Text GLabel 6600 900  2    60   Input ~ 0
 VCC
 $Comp
 L R R10
 U 1 1 53055831
-P 7000 1600
-F 0 "R10" V 7080 1600 40  0000 C CNN
-F 1 "3M" V 7007 1601 40  0000 C CNN
-F 2 "~" V 6930 1600 30  0000 C CNN
-F 3 "~" H 7000 1600 30  0000 C CNN
-	1    7000 1600
+P 6250 1650
+F 0 "R10" V 6330 1650 40  0000 C CNN
+F 1 "3M" V 6257 1651 40  0000 C CNN
+F 2 "~" V 6180 1650 30  0000 C CNN
+F 3 "~" H 6250 1650 30  0000 C CNN
+	1    6250 1650
 	1    0    0    -1
 $EndComp
@@
 L GND #PWR11
 U 1 1 53055869
-P 7000 1950
-F 0 "#PWR11" H 7000 1950 30  0001 C CNN
-F 1 "GND" H 7000 1880 30  0001 C CNN
-F 2 "" H 7000 1950 60  0000 C CNN
-F 3 "" H 7000 1950 60  0000 C CNN
-	1    7000 1950
+P 6250 2000
+F 0 "#PWR11" H 6250 2000 30  0001 C CNN
+F 1 "GND" H 6250 1930 30  0001 C CNN
+F 2 "" H 6250 2000 60  0000 C CNN
+F 3 "" H 6250 2000 60  0000 C CNN
+	1    6250 2000
 	1    0    0    -1
 $EndComp
@@
 Text GLabel 7250 6100 0    60   Input ~ 0
 USER_SW
-Text Notes 1550 4750 0    60   ~ 0
-weak pulldown to\nstart LPS. I/O\nstates are preserved\nthrough sleep mode.
-$Comp
-L R R1
-U 1 1 530F3C34
-P 1400 4550
-F 0 "R1" V 1480 4550 40  0000 C CNN
-F 1 "3M" V 1407 4551 40  0000 C CNN
-F 2 "~" V 1330 4550 30  0000 C CNN
-F 3 "~" H 1400 4550 30  0000 C CNN
-	1    1400 4550
-	1    0    0    -1
-$EndComp
+Text Notes 1400 4000 0    60   ~ 0
+weak pullup to\nstart LPS. I/O\nstates are preserved\nthrough sleep mode.
 Text Notes 1100 7300 0    60   ~ 0
 NP- optional accessory\npower control
 Text Notes 5550 7400 0    60   ~ 0
 NP- accessory\nexpansion\nheader
-$Comp
-L GND #PWR1
-U 1 1 530F3C3A
-P 1400 4900
-F 0 "#PWR1" H 1400 4900 30  0001 C CNN
-F 1 "GND" H 1400 4830 30  0001 C CNN
-F 2 "" H 1400 4900 60  0000 C CNN
-F 3 "" H 1400 4900 60  0000 C CNN
-	1    1400 4900
-	1    0    0    -1
-$EndComp
-$Comp
-L MOSFET_N Q2
-U 1 1 5355278E
-P 2050 4200
-F 0 "Q2" H 2050 4000 60  0000 R CNN
-F 1 "MOSFET_N" H 2050 4400 60  0000 R CNN
-F 2 "~" H 2050 4200 60  0000 C CNN
-F 3 "~" H 2050 4200 60  0000 C CNN
-	1    2050 4200
-	1    0    0    -1
-$EndComp
 Text GLabel 6700 4350 2    60   Input ~ 0
 USER_SW
@@
 	4850 4050 4950 4050
 Wire Wire Line
-	2400 3900 2150 3900
-Wire Wire Line
-	2150 3800 2150 4000
-Connection ~ 2150 3900
-Wire Wire Line
-	1150 4200 1850 4200
-Wire Wire Line
-	2150 3200 2150 3300
-Wire Wire Line
-	2150 4500 2150 4400
+	2350 4450 2550 4450
+Wire Wire Line
+	2450 3750 2450 3850
 Wire Wire Line
 	8750 1050 8850 1050
@@
 	9850 1500 9750 1500
 Wire Wire Line
-	7350 950  7350 1050
-Wire Wire Line
-	6950 1250 7050 1250
-Wire Wire Line
-	7350 1550 7350 1450
-Wire Wire Line
-	7000 1350 7000 1250
-Connection ~ 7000 1250
-Wire Wire Line
-	7000 1950 7000 1850
+	6600 900  6600 1100
+Wire Wire Line
+	6200 1300 6300 1300
+Wire Wire Line
+	6600 1500 6600 1750
+Wire Wire Line
+	6250 1400 6250 1300
+Connection ~ 6250 1300
+Wire Wire Line
+	6250 2000 6250 1900
 Wire Wire Line
 	5550 5250 5550 5150
@@
 	1600 5500 1500 5500
 Wire Wire Line
-	2050 3200 2150 3200
-Connection ~ 1400 4200
+	2350 3750 2450 3750
 Wire Notes Line
 	800  5800 2600 5800
@@
 Wire Notes Line
 	6250 6250 5450 6250
-Wire Wire Line
-	1400 4300 1400 4200
-Wire Wire Line
-	1400 4900 1400 4800
 $Comp
 L R R?
@@
 	9350 4550 9350 4450
 Wire Wire Line
-	9350 3950 9350 3850
+	9350 3850 9350 3950
 Wire Wire Line
 	9350 3350 9350 3250
@@
 Text GLabel 9100 4100 0    60   Input ~ 0
 VFB_SNS/USB_SNS
+Wire Wire Line
+	2450 4450 2450 4350
+Connection ~ 2450 4450
+$Comp
+L R R?
+U 1 1 5356CEC2
+P 7000 1300
+F 0 "R?" V 7080 1300 40  0000 C CNN
+F 1 "0R" V 7007 1301 40  0000 C CNN
+F 2 "~" V 6930 1300 30  0000 C CNN
+F 3 "~" H 7000 1300 30  0000 C CNN
+	1    7000 1300
+	1    0    0    -1
+$EndComp
+Connection ~ 6600 1000
+Connection ~ 6600 1600
+Wire Wire Line
+	6600 1000 7000 1000
+Wire Wire Line
+	7000 1000 7000 1050
+Wire Wire Line
+	7000 1550 7000 1600
+Wire Wire Line
+	7000 1600 6600 1600
+Text Notes 7200 1450 0    60   ~ 0
+nopop
 $EndSCHEMATC
